Commit message: feat: add gazebo world and proper URDF parameters

File: franka_description/robots/panda_arm.urdf.xacro (robot description, xacro)
@@ -1,5 +1,10 @@
-<?xml version='1.0' encoding='utf-8'?>
-<robot xmlns:xacro="http://www.ros.org/wiki/xacro" name="panda">
-  <xacro:include filename="$(find franka_description)/robots/panda_arm.xacro" />
-  <xacro:panda_arm />
+<?xml version="1.0" encoding="utf-8"?>
+<robot xmlns:xacro="http://www.ros.org/wiki/xacro" name="panda_arm">
+  <xacro:arg name="hardware_interface" default="PositionJointInterface"/>
+  <xacro:arg name="robot_name" default="panda"/>
+  <xacro:arg name="parent" default='world'/>
+  <xacro:include filename="$(find franka_description)/robots/panda_arm/panda_arm.xacro"/>
+  <xacro:panda_arm robot_name="$(arg robot_name)" parent="$(arg parent)" hardware_interface="$(arg hardware_interface)">
+  	<origin xyz="0 0 0" rpy="0 0 0"/>
+  </xacro:panda_arm>
 </robot>

File: franka_description/robots/panda_arm_hand.urdf.xacro (robot description, xacro)
@@ -1,7 +1,38 @@
 <?xml version="1.0" encoding="utf-8"?>
 <robot xmlns:xacro="http://www.ros.org/wiki/xacro" name="panda">
-  <xacro:include filename="$(find franka_description)/robots/panda_arm.xacro"/>
-  <xacro:include filename="$(find franka_description)/robots/hand.xacro"/>
-  <xacro:panda_arm />
-  <xacro:hand ns="panda" rpy="0 0 ${-pi/4}" connected_to="panda_link8"/>
+  <xacro:arg name="hardware_interface" default="PositionJointInterface"/>
+  <xacro:arg name="robot_name" default="panda"/>
+  <xacro:arg name="parent" default=''/>
+  <xacro:include filename="$(find franka_description)/robots/panda_arm/panda_arm.xacro"/>
+  <!-- <xacro:include filename="$(find franka_description)/robots/panda_hand/hand.xacro"/> -->
+	<xacro:property name="parent_" value="$(arg parent)" />
+	<!-- <xacro:unless value="${not $(arg parent)}">			</xacro:unless> -->
+	<xacro:if value="${not parent_}">
+		<xacro:property name="parent_" value="world" />
+    <link name="${parent_}">
+        <visual>
+            <geometry>
+                <box size="2. 2 0.01"/>
+            </geometry>
+            <origin xyz="0 0 0"/>
+        </visual>
+        <collision>
+            <geometry>
+                <box size="2. 2 0.01"/>
+            </geometry>
+            <origin xyz="0 0 0"/>
+        </collision>
+        <intertial>
+            <mass value="100"/>
+            <inertia ixx="8" ixy="0" ixz="0" iyy="8" iyz="0" izz="8"/>
+        </intertial>
+    </link>
+		<gazebo reference="world">
+		    <static>true</static>
+		</gazebo>
+	</xacro:if>
+  <xacro:panda_arm robot_name="$(arg robot_name)" parent="${parent_}" hardware_interface="$(arg hardware_interface)">
+  	<origin xyz="0 0 0" rpy="0 0 0"/>
+  </xacro:panda_arm>
+  <xacro:hand ns="${robot_name}" rpy="0 0 ${-pi/4}" connected_to="panda_link8"/>
 </robot>
