Commit message: feat: launch franka_common franka_moveit launch the franka in gazebo and start moveit

File: franka_description/robots/arm_base/arm_base.xacro (robot description, xacro)
@@ -2,5 +2,5 @@
 <robot xmlns:xacro="http://www.ros.org/wiki/xacro">
   <xacro:property name="M_PI" value="3.1415926535897931" />
-  <xacro:include filename="$(find franka_world)/urdf/arm_base/arm_base.gazebo.xacro" />
+  <xacro:include filename="$(find franka_description)/robots/arm_base/arm_base.gazebo.xacro" />
   <xacro:macro name="arm_base" params="parent base_adapter_child">
     <joint name="table_joint" type="fixed">
@@ -18,5 +18,5 @@
         <origin xyz="0 0 0" rpy="0 0 ${90 * pi / 180}"/>
         <geometry>
-          <mesh filename="package://franka_world/meshes/arm_base/visual/table.dae"/>
+          <mesh filename="package://franka_description/meshes/arm_base/visual/table.dae"/>
         </geometry>
       </visual>
@@ -40,5 +40,5 @@
         <origin xyz="0 0 0" rpy="0 0 0"/>
         <geometry>
-          <mesh filename="package://franka_world/meshes/arm_base/visual/base_adapter.dae"/>
+          <mesh filename="package://franka_description/meshes/arm_base/visual/base_adapter.dae"/>
         </geometry>
       </visual>

File: franka_description/robots/panda_arm/panda_arm.xacro (robot description, xacro)
@@ -16,5 +16,5 @@
   <xacro:macro name="panda_arm" params="robot_name parent hardware_interface *origin">
     <!--joint between {parent} and link_0-->
-    <joint name="${parent}_${robot_name}_joint" type="fixed">
+    <joint name="${robot_name}_joint0" type="fixed">
       <xacro:insert_block name="origin"/>
       <parent link="${parent}"/>

File: franka_moveit_config/config/panda_arm.srdf.xacro (robot description, xacro)
@@ -4,6 +4,6 @@
     A URDF file must exist for this robot as well, where the joints and the links that are referenced are defined
 -->
-<robot xmlns:xacro="http://www.ros.org/wiki/xacro" name="panda">
-  <xacro:include filename="$(find panda_moveit_config)/config/panda_arm.xacro" />
+<robot xmlns:xacro="http://www.ros.org/wiki/xacro" name="panda_arm">
+  <xacro:include filename="$(find franka_moveit_config)/config/panda_arm.xacro" />
   <xacro:panda_arm />
 </robot>

File: franka_moveit_config/config/panda_arm.xacro (robot description, xacro)
@@ -1,4 +1,4 @@
 <?xml version="1.0" ?>
-<robot xmlns:xacro="http://www.ros.org/wiki/xacro" name="panda">
+<robot xmlns:xacro="http://www.ros.org/wiki/xacro" name="panda_arm">
   <xacro:macro name="panda_arm">
     <!--GROUPS: Representation of a set of joints and links. This can be useful for specifying DOF to plan for, defining arms, end effectors, etc-->
@@ -20,7 +20,34 @@
       <joint name="panda_joint7" value="0.785" />
     </group_state>
+    <group_state name="home" group="panda_arm">
+        <joint name="panda_joint1" value="0" />
+        <joint name="panda_joint2" value="0" />
+        <joint name="panda_joint3" value="0" />
+        <joint name="panda_joint4" value="-1.5707" />
+        <joint name="panda_joint5" value="0" />
+        <joint name="panda_joint6" value="1.5707" />
+        <joint name="panda_joint7" value="0" />
+    </group_state>
+    <group_state name="home_up" group="panda_arm">
+        <joint name="panda_joint1" value="0" />
+        <joint name="panda_joint2" value="0" />
+        <joint name="panda_joint3" value="0" />
+        <joint name="panda_joint4" value="0" />
+        <joint name="panda_joint5" value="0" />
+        <joint name="panda_joint6" value="3.1415" />
+        <joint name="panda_joint7" value="0" />
+    </group_state>
+    <group_state name="folded" group="panda_arm">
+        <joint name="panda_joint1" value="0" />
+        <joint name="panda_joint2" value="0" />
+        <joint name="panda_joint3" value="0" />
+        <joint name="panda_joint4" value="-2.9222" />
+        <joint name="panda_joint5" value="0.032" />
+        <joint name="panda_joint6" value="0.0349" />
+        <joint name="panda_joint7" value="-2.2" />
+    </group_state>
     <!--END EFFECTOR: Purpose: Represent information about an end effector.-->
     <!--VIRTUAL JOINT: Purpose: this element defines a virtual joint between a robot link and an external frame of reference (considered fixed with respect to the robot)-->
-    <virtual_joint name="virtual_joint" type="floating" parent_frame="world" child_link="panda_link0" />
+    <!-- <virtual_joint name="virtual_joint" type="floating" parent_frame="world" child_link="panda_link0" /> -->
     <!--DISABLE COLLISIONS: By default it is assumed that any link of the robot could potentially come into collision with any other link in the robot. This tag disables collision checking between a specified pair of links. -->
     <disable_collisions link1="panda_link0" link2="panda_link1" reason="Adjacent" />

File: franka_moveit_config/config/panda_arm_hand.srdf.xacro (robot description, xacro)
@@ -4,5 +4,5 @@
     A URDF file must exist for this robot as well, where the joints and the links that are referenced are defined
 -->
-<robot xmlns:xacro="http://www.ros.org/wiki/xacro" name="panda">
+<robot xmlns:xacro="http://www.ros.org/wiki/xacro" name="panda_arm">
   <xacro:include filename="$(find panda_moveit_config)/config/panda_arm.xacro" />
   <xacro:include filename="$(find panda_moveit_config)/config/hand.xacro" />

Commit message: chore: more extensible file description structure

File: franka_description/robots/arm_base/arm_base.xacro (robot description, xacro)
@@ -3,4 +3,5 @@
   <xacro:property name="M_PI" value="3.1415926535897931" />
   <xacro:include filename="$(find franka_description)/robots/arm_base/arm_base.gazebo.xacro" />
+  <xacro:include filename="$(find franka_description)/robots/materials.xacro" />
   <xacro:macro name="arm_base" params="parent base_adapter_child">
     <joint name="table_joint" type="fixed">
@@ -34,17 +35,23 @@
       <parent link="table" />
       <child link="${base_adapter_child}" />
-      <origin xyz="-0.2 0 0" rpy="0 0 0"/>
+      <origin xyz="-0.38 0 0.025" rpy="0 0 0"/>
     </joint>
     <link name="${base_adapter_child}">
       <visual>
-        <origin xyz="0 0 0" rpy="0 0 0"/>
+        <material name="grey"/>
+        <origin xyz="-0.072 0 -0.0125" rpy="0 0 0"/>
         <geometry>
-          <mesh filename="package://franka_description/meshes/arm_base/visual/base_adapter.dae"/>
+          <box size="0.3 0.3 0.025" />
+          <!-- <mesh filename="package://franka_description/meshes/arm_base/visual/base_adapter.dae"/> -->
         </geometry>
       </visual>
       <collision>
-        <origin xyz="0 0 0.01" rpy="0 0 0"/>
+        <origin xyz="-0.072 0 -0.0125" rpy="0 0 0"/>
         <geometry>
-          <cylinder length="0.02" radius="0.16"/>
+          <!-- Real box dimension -->
+          <!-- <box size="0.4 0.4 0.025" /> -->
+          <!-- Augmented box dimension -->
+          <box size="0.4 0.4 0.3" />
+          <!-- <cylinder length="0.02" radius="0.16"/> -->
         </geometry>
       </collision>

File: franka_description/robots/panda_arm/panda_arm.xacro (robot description, xacro)
@@ -14,5 +14,5 @@
   <!-- TODO: set the correct individual effort values for every joint -->
   <xacro:property name="max_effort" value="300"/>
-  <xacro:macro name="panda_arm" params="robot_name parent hardware_interface *origin">
+  <xacro:macro name="panda_arm" params="hand_link_name=:'' robot_name parent hardware_interface *origin">
     <!--joint between {parent} and link_0-->
     <joint name="${robot_name}_joint0" type="fixed">
@@ -285,4 +285,11 @@
       </inertial>
     </link>
+    <xacro:if value="${not hand_link_name}">
+      <joint name="${robot_name}_hand_joint" type="fixed">
+        <parent link="${robot_name}_link8"/>
+        <child link="$(arg robot_name)_hand"/>
+        <origin xyz="0 0 0" rpy="0 0 ${-pi/4}"/>
+      </joint>
+    </xacro:if>
     <!--Extensions -->
     <xacro:panda_gazebo robot_name="${robot_name}" />

File: franka_description/robots/panda_arm_hand.urdf.xacro (robot description, xacro)
@@ -3,36 +3,32 @@
   <xacro:arg name="hardware_interface" default="PositionJointInterface"/>
   <xacro:arg name="robot_name" default="panda"/>
-  <xacro:arg name="parent" default=''/>
   <xacro:include filename="$(find franka_description)/robots/panda_arm/panda_arm.xacro"/>
-  <!-- <xacro:include filename="$(find franka_description)/robots/panda_hand/hand.xacro"/> -->
-	<xacro:property name="parent_" value="$(arg parent)" />
+  <xacro:include filename="$(find franka_description)/robots/panda_hand/panda_hand.xacro"/>
 	<!-- <xacro:unless value="${not $(arg parent)}">			</xacro:unless> -->
-	<xacro:if value="${not parent_}">
-		<xacro:property name="parent_" value="world" />
-    <link name="${parent_}">
-        <visual>
-            <geometry>
-                <box size="2. 2 0.01"/>
-            </geometry>
-            <origin xyz="0 0 0"/>
-        </visual>
-        <collision>
-            <geometry>
-                <box size="2. 2 0.01"/>
-            </geometry>
-            <origin xyz="0 0 0"/>
-        </collision>
-        <intertial>
-            <mass value="100"/>
-            <inertia ixx="8" ixy="0" ixz="0" iyy="8" iyz="0" izz="8"/>
-        </intertial>
-    </link>
-		<gazebo reference="world">
-		    <static>true</static>
-		</gazebo>
-	</xacro:if>
-  <xacro:panda_arm robot_name="$(arg robot_name)" parent="${parent_}" hardware_interface="$(arg hardware_interface)">
+	<xacro:property name="parent_" value="world" />
+  <link name="${parent_}">
+      <visual>
+          <geometry>
+              <box size="2. 2 0.01"/>
+          </geometry>
+          <origin xyz="0 0 0"/>
+      </visual>
+      <collision>
+          <geometry>
+              <box size="2. 2 0.01"/>
+          </geometry>
+          <origin xyz="0 0 0"/>
+      </collision>
+      <intertial>
+          <mass value="100"/>
+          <inertia ixx="8" ixy="0" ixz="0" iyy="8" iyz="0" izz="8"/>
+      </intertial>
+  </link>
+	<gazebo reference="world">
+	    <static>true</static>
+	</gazebo>
+  <xacro:panda_arm robot_name="$(arg robot_name)" parent="${parent_}" hardware_interface="$(arg hardware_interface)" hand_link_name="$(arg robot_name)_hand">
   	<origin xyz="0 0 0" rpy="0 0 0"/>
   </xacro:panda_arm>
-  <xacro:hand ns="${robot_name}" rpy="0 0 ${-pi/4}" connected_to="panda_link8"/>
+  <xacro:panda_hand robot_name="$(arg robot_name)" hardware_interface="$(arg hardware_interface)" first_link_name="$(arg robot_name)_hand"/>
 </robot>

File: franka_description/robots/panda_arm_on_table.urdf.xacro (robot description, xacro)
@@ -3,23 +3,13 @@
   <xacro:arg name="hardware_interface" default="PositionJointInterface"/>
   <xacro:arg name="robot_name" default="panda"/>
-  <xacro:arg name="parent" default=''/>
-  <xacro:include filename="$(find franka_description)/robots/panda_arm/panda_arm.xacro"/>
-  <xacro:include filename="$(find franka_description)/robots/arm_base/arm_base.xacro"/>
-  <xacro:property name="parent_" value="$(arg parent)" />
-  <xacro:if value="${not parent_}">
-    <xacro:property name="parent_" value="world" />
-    <link name="${parent_}">
-    	<intertial>
-  	    <mass value="100"/>
-      <inertia ixx="8" ixy="0" ixz="0" iyy="8" iyz="0" izz="8"/>
-    	</intertial>
-    </link>
-    <gazebo reference="${parent_}">
-        <static>true</static>
-    </gazebo>
-  </xacro:if>
-  <xacro:arm_base parent="${parent_}" base_adapter_child="$(arg robot_name)_base"/>
-  <xacro:panda_arm robot_name="$(arg robot_name)" parent="$(arg robot_name)_base" hardware_interface="$(arg hardware_interface)">
-  	<origin xyz="0 0 0.02" rpy="0 0 0"/> <!-- TODO: this offset should be inside the arm_base -->
-  </xacro:panda_arm>
+  <xacro:arg name="hand_link_name" default=''/>
+  <xacro:arg name="hand_link_name" default=''/>
+  <xacro:include filename="$(find franka_description)/robots/arm_table.xacro"/>
+  <xacro:property name="parent" value="world" />
+  <link name="${parent}"/>
+  <gazebo reference="${parent}">
+      <static>true</static>
+  </gazebo>
+  <!-- hand_link_name=:''  -->
+  <xacro:arm_hand_table parent="${parent}" robot_name="$(arg robot_name)" hardware_interface="$(arg hardware_interface)"/>
 </robot>

File: franka_description/robots/panda_hand/panda_hand.xacro (robot description, xacro)
@@ -1,15 +1,10 @@
 <?xml version="1.0"?>
 <robot xmlns:xacro="http://www.ros.org/wiki/xacro">
-  <xacro:include filename="$(find franka_description)/urdf/franka_hand/franka_hand.gazebo.xacro"/>
-  <xacro:include filename="$(find franka_description)/urdf/franka_hand/franka_hand.transmission.xacro"/>
+  <xacro:include filename="$(find franka_description)/robots/panda_hand/panda_hand.gazebo.xacro"/>
+  <xacro:include filename="$(find franka_description)/robots/panda_hand/panda_hand.transmission.xacro"/>
   <xacro:property name="joint_lower_limit" value="0.0" />
   <xacro:property name="joint_upper_limit" value="0.055" />
-  <xacro:macro name="franka_hand" params="parent hardware_interface robot_name">
-    <joint name="${parent}_hand_joint" type="fixed">
-      <parent link="${parent}"/>
-      <child link="${robot_name}_hand"/>
-      <origin xyz="0 0 0" rpy="0 0 ${-pi/4}"/>
-    </joint>
-    <link name="${robot_name}_hand">
+  <xacro:macro name="panda_hand" params="robot_name hardware_interface first_link_name">
+    <link name="${first_link_name}">
       <inertial>
         <mass value="0.73" />
@@ -20,5 +15,5 @@
         <origin xyz="0 0 0" rpy="0 0 0"/>
         <geometry>
-          <mesh filename="package://franka_description/meshes/franka_hand/visual/hand.dae"/>
+          <mesh filename="package://franka_description/meshes/panda_hand/visual/hand.dae"/>
         </geometry>
         <material name="">
@@ -29,5 +24,5 @@
         <origin xyz="0 0 0" rpy="0 0 0"/>
         <geometry>
-          <mesh filename="package://franka_description/meshes/franka_hand/collision/hand.stl"/>
+          <mesh filename="package://franka_description/meshes/panda_hand/collision/hand.stl"/>
         </geometry>
       </collision>
@@ -49,5 +44,5 @@
         <origin xyz="0 0 0" rpy="0 0 0"/>
         <geometry>
-          <mesh filename="package://franka_description/meshes/franka_hand/visual/finger.dae"/>
+          <mesh filename="package://franka_description/meshes/panda_hand/visual/finger.dae"/>
         </geometry>
         <material name="">
@@ -58,5 +53,5 @@
         <origin xyz="0 0 0" rpy="0 0 0"/>
         <geometry>
-          <mesh filename="package://franka_description/meshes/franka_hand/collision/finger.stl"/>
+          <mesh filename="package://franka_description/meshes/panda_hand/collision/finger.stl"/>
         </geometry>
       </collision>
@@ -78,5 +73,5 @@
         <origin xyz="0 0 0" rpy="0 0 ${pi}"/>
         <geometry>
-          <mesh filename="package://franka_description/meshes/franka_hand/visual/finger.dae"/>
+          <mesh filename="package://franka_description/meshes/panda_hand/visual/finger.dae"/>
         </geometry>
         <material name="">
@@ -87,10 +82,10 @@
         <origin xyz="0 0 0" rpy="0 0 ${pi}"/>
         <geometry>
-          <mesh filename="package://franka_description/meshes/franka_hand/collision/finger.stl"/>
+          <mesh filename="package://franka_description/meshes/panda_hand/collision/finger.stl"/>
         </geometry>
       </collision>
     </link>
-    <xacro:franka_hand_gazebo robot_name="${robot_name}" />
-    <xacro:franka_hand_transmission hardware_interface="${hardware_interface}" robot_name="${robot_name}"/>
+    <xacro:panda_hand_gazebo robot_name="${robot_name}" />
+    <xacro:panda_hand_transmission hardware_interface="${hardware_interface}" robot_name="${robot_name}"/>
   </xacro:macro>
 </robot>

File: franka_moveit_config/config/panda_arm_hand.srdf.xacro (robot description, xacro)
@@ -35,5 +35,5 @@
   <disable_collisions link1="panda_hand" link2="panda_link6" reason="Never" />
   <disable_collisions link1="panda_hand" link2="panda_link7" reason="Adjacent" />
-  <disable_collisions link1="panda_leftfinger" link2="panda_link3" reason="Never" />
+  <!-- <disable_collisions link1="panda_leftfinger" link2="panda_link3" reason="Never" />
   <disable_collisions link1="panda_leftfinger" link2="panda_link4" reason="Never" />
   <disable_collisions link1="panda_leftfinger" link2="panda_link6" reason="Never" />
@@ -42,4 +42,4 @@
   <disable_collisions link1="panda_link4" link2="panda_rightfinger" reason="Never" />
   <disable_collisions link1="panda_link6" link2="panda_rightfinger" reason="Never" />
-  <disable_collisions link1="panda_link7" link2="panda_rightfinger" reason="Never" />
+  <disable_collisions link1="panda_link7" link2="panda_rightfinger" reason="Never" /> -->
 </robot>
